File: pcb/WerfenMc/WerfenMc_power_edit.kicad_pcb (KiCad board)
At the start: 2 copper layers, 72 x 57 mm, 71 parts, among them J1 MOTOR, J2 SWD, J3 POWER, J4 UART3, J5 UART1, J6 PowerTerminal, Q1 Q_Photo_NPN, Q2 BCP56, SW1 RESET, SW2 ESTOP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

Commit message: Reverse engineer the actual layout with the new schottkey (whoops)
Parts:
- D8: footprint Diode_SMD:D_0805_2012Metric -> Diode_SMD:D_SMC
- moved C14 15.3 mm to (85.8, 48.2), turned to -90 degrees
- moved D10 7.84 mm to (92.8, 45.7), turned to 180 degrees
- moved R17 4.46 mm to (92.3, 47.5), turned to 180 degrees
- moved D8 3.99 mm to (80.8, 33.8), turned to 0 degrees
- moved R10 2.99 mm to (94.0, 81.2)
- moved C15 2.49 mm to (56.4, 35.8)
- moved TP3 1.92 mm to (83.1, 40.5)
- moved A1 1.86 mm to (102.0, 56.4)
- moved R8 1.80 mm to (84.2, 71.8)
- moved L1 1.69 mm to (68.8, 32.8)
- moved TP2 1.69 mm to (54.8, 45.0)
- moved TP8 1.69 mm to (66.3, 39.8)
- moved U2 1.69 mm to (74.9, 46.8)
- moved U3 1.69 mm to (61.9, 45.0)
- moved J1 1.68 mm to (94.6, 52.4)
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Routing:
- net +3.3V: track 199.8 -> 209.2 mm
- net +12V: track 33.1 -> 28.9 mm
- net +5V: track 31.3 -> 28.8 mm
- net Net-(D5-Pad2): track 19.2 -> 16.9 mm
- net Net-(D5-Pad1): track 1.96 -> 3.23 mm
- net 2B: track 13.3 -> 14.3 mm
- net MS1: track 23.9 -> 24.7 mm
- net MS2: track 27.5 -> 28.3 mm
- net MS3: track 30.3 -> 31.1 mm
- net DIR: track 38.3 -> 39.1 mm
- net 1A: track 10.3 -> 11.1 mm
- net ENABLE: track 21.2 -> 21.9 mm
- net GND: track 112.9 -> 113.6 mm, vias 52 -> 48
- net 2A: track 4.55 -> 5.14 mm
Other:
- board text removed: "PWR"
