File: pcb/WerfenMc/WerfenMc_power_edit.kicad_sch (KiCad schematic)
At the start: 71 parts, among them J1 MOTOR, J2 SWD, J3 POWER, J4 UART3, J5 UART1, J6 PowerTerminal, Q1 Q_Photo_NPN, Q2 BCP56, SW1 RESET, SW2 ESTOP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

Commit message: Reverse engineer the actual layout with the new schottkey (whoops)
Parts:
- D8: footprint Diode_SMD:D_0805_2012Metric -> Diode_SMD:D_SMC
Changed lines of the file:
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@@
       (effects (font (size 1.27 1.27)) (justify right))
     )
-    (property "Footprint" "Diode_SMD:D_0805_2012Metric" (id 2) (at 214.63 137.16 0)
+    (property "Footprint" "Diode_SMD:D_SMC" (id 2) (at 214.63 137.16 0)
       (effects (font (size 1.27 1.27)) hide)
     )
@@
     )
     (path "/c3e73251-33aa-40ec-b69f-04b50752ec99"
-      (reference "D8") (unit 1) (value "D_Schottky") (footprint "Diode_SMD:D_0805_2012Metric")
+      (reference "D8") (unit 1) (value "D_Schottky") (footprint "Diode_SMD:D_SMC")
     )
     (path "/2e86fc63-f29e-4dc1-b1d0-9e149bbee12b"
